File: PHM-30A/PHM-30A.kicad_pcb (KiCad board)
At the start: 2 copper layers, 0 parts

Commit message: Modificado el part number de D1 y D2 Modificado el Footprint del Gyroscopio para marcar el pin 1 en el silkscreen
Parts:
- added C1: C, Capacitor_SMD:C_0805_2012Metric, F.Cu at (169.1, 58.2)
- added C2: C, Capacitor_SMD:C_0805_2012Metric, F.Cu at (164.0, 58.2)
- added C3: C, Capacitor_SMD:C_0805_2012Metric, F.Cu at (160.3, 58.2)
- added C4: C, Capacitor_SMD:C_0805_2012Metric, F.Cu at (173.7, 58.2)
- added C5: C, Capacitor_SMD:C_0603_1608Metric, F.Cu at (160.9, 46.5)
- added C6: C, Capacitor_SMD:C_0603_1608Metric, F.Cu at (173.9, 46.5)
- added J1: Conn_01x04_Socket, Connector_PinSocket_1.27mm:PinSocket_1x04_P1.27mm_Castellated, F.Cu at (165.7, 85.1)
- added J2: Conn_01x04_Socket, Connector_PinSocket_1.27mm:PinSocket_1x04_P1.27mm_Castellated, F.Cu at (176.7, 64.0)
- added J3: Conn_01x04_Socket, Connector_PinSocket_1.27mm:PinSocket_1x04_P1.27mm_Castellated, F.Cu at (176.7, 71.6)
- added J4: Conn_01x04_Socket, Connector_PinSocket_1.27mm:PinSocket_1x04_P1.27mm_Castellated, F.Cu at (158.1, 67.9)
- added J5: Conn_01x04_Socket, Connector_PinSocket_1.27mm:PinSocket_1x04_P1.27mm_Castellated, F.Cu at (158.4, 61.0)
- added J6: Conn_01x04_Socket, Connector_PinSocket_1.27mm:PinSocket_1x04_P1.27mm_Castellated, F.Cu at (176.7, 55.9)
- added J7: Conn_01x04_Socket, Connector_PinSocket_1.27mm:PinSocket_1x04_P1.27mm_Castellated, F.Cu at (158.1, 52.1)
- added Q1: QM6006D, Package_TO_SOT_SMD:TO-252-2, F.Cu at (171.0, 68.5)
- added Q2: QM6006D, Package_TO_SOT_SMD:TO-252-2, F.Cu at (163.8, 80.0)
- added Q3: QM6006D, Package_TO_SOT_SMD:TO-252-2, F.Cu at (163.9, 68.5)
- added Q5: QM6006D, Package_TO_SOT_SMD:TO-252-2, F.Cu at (171.0, 80.0)
- added R1: R_US, Resistor_SMD:R_0603_1608Metric, F.Cu at (164.5, 46.5)
- added R2: R_US, Resistor_SMD:R_0603_1608Metric, F.Cu at (169.3, 46.5)
- added U1: L6491, Package_SO:SO-14_3.9x8.65mm_P1.27mm, F.Cu at (171.3, 52.1)
- added U2: L6491, Package_SO:SO-14_3.9x8.65mm_P1.27mm, F.Cu at (163.4, 52.1)
Routing:
- added copper zone on F.Cu, net /VH
- added copper zone on F.Cu, net GND
Other:
- board outline added: 18.5 x 40 mm
