File: PHM-30A/PHM-30A.kicad_sch (KiCad schematic)
At the start: 0 parts

Commit message: Modificado el part number de D1 y D2 Modificado el Footprint del Gyroscopio para marcar el pin 1 en el silkscreen
Parts:
- added C1, C2, C3, C4: C, Capacitor_SMD:C_0805_2012Metric, symbol Device:C
- added C5, C6: C, Capacitor_SMD:C_0603_1608Metric, symbol Device:C
- added J1, J2, J3, J4, J5, J6, J7: Conn_01x04_Socket, Connector_PinSocket_1.27mm:PinSocket_1x04_P1.27mm_Castellated, symbol Connector:Conn_01x04_Socket
- added Q1, Q2, Q3, Q5: QM6006D, Package_TO_SOT_SMD:TO-252-2, symbol Transistor_FET:QM6006D
- added R1, R2: R_US, Resistor_SMD:R_0603_1608Metric, symbol Device:R_US
- added U1, U2: L6491, Package_SO:SO-14_3.9x8.65mm_P1.27mm, symbol Driver_FET:L6491
Connections:
- new net: Q2.1 (G), U2.13 (HVG)
- new net: C3.1, U2.14 (BOOT)
- new net: C5.2, R1.1, U2.5 (DT)
- new net: Q3.1 (G), U2.8 (LVG)
- new net: C6.2, R2.1, U1.5 (DT)
- new net: Q1.1 (G), U1.8 (LVG)
- new net: Q5.1 (G), U1.13 (HVG)
- new net: C1.1, U1.14 (BOOT)
- new net A: C1.2, J3.1 (Pin_1), J3.2 (Pin_2), J3.3 (Pin_3), J3.4 (Pin_4), Q1.2 (D), Q5.3 (S), U1.12 (OUT)
- new net B: C3.2, J4.1 (Pin_1), J4.2 (Pin_2), J4.3 (Pin_3), J4.4 (Pin_4), Q2.3 (S), Q3.2 (D), U2.12 (OUT)
- new net GND: C2.2, C4.1, C5.1, C6.1, J2.1 (Pin_1), J2.2 (Pin_2), J2.3 (Pin_3), J2.4 (Pin_4), J5.1 (Pin_1), J5.2 (Pin_2), J5.3 (Pin_3), J5.4 (Pin_4), Q1.3 (S), Q3.3 (S), R1.2, R2.2, U1.6 (SGND), U1.7 (PGND), U2.6 (SGND), U2.7 (PGND)
- new net HIN_D: J7.1 (Pin_1), U2.3 (HIN)
- new net HIN_I: J6.3 (Pin_3), U1.3 (HIN)
- new net LIN_D: J7.3 (Pin_3), U2.1 (~{LIN})
- new net LIN_I: J6.1 (Pin_1), U1.1 (~{LIN})
- new net SD_D: J7.2 (Pin_2), U2.2 (~{SD}/OD)
- new net SD_I: J6.2 (Pin_2), U1.2 (~{SD}/OD)
- new net VCC: C2.1, C4.2, J6.4 (Pin_4), J7.4 (Pin_4), U1.4 (VCC), U2.4 (VCC)
- new net VH: J1.1 (Pin_1), J1.2 (Pin_2), J1.3 (Pin_3), J1.4 (Pin_4), Q2.2 (D), Q5.2 (D)
